Commit message: Obstacle Gazebo world

File: autorally_description/urdf/autoRallyPlatform.urdf.xacro (robot description, xacro)
@@ -410,4 +410,12 @@
       <inertia ixx="1e-6" ixy="0" ixz="0" iyy="1e-6" iyz="0" izz="1e-6" />
     </inertial>
+  </link>
+  <!-- Reference frame for left camera (for stereo camera)-->
+  <joint name="left_camera_optical_joint" type="fixed">
+    <origin xyz="0 0.07 0" rpy="0 0 0"/>
+    <parent link="camera_link"/>
+    <child link="left_camera_optical_frame"/>
+  </joint>
+  <link name="left_camera_optical_frame">
   </link>
   <!-- camera -->

Commit message: Collision detection

File: autorally_description/urdf/autoRallyPlatform.urdf.xacro (robot description, xacro)
@@ -324,5 +324,5 @@
       </geometry>
     </visual>
-    <collision>
+    <collision name="chassis_collision">
       <origin xyz="${-chassis_length/2 + 0.2} 0 ${-chassis_cm_height}"
               rpy="0 0 0"/>

Commit message: LIDAR integration and increased laser retroreflector for obstacels

File: autorally_description/urdf/autoRallyPlatform.urdf.xacro (robot description, xacro)
@@ -315,4 +315,9 @@
     <material>Gazebo/Grey</material>
   </gazebo>
+  <!-- Velodyne LIDAR -->
+  <xacro:include filename="$(find velodyne_description)/urdf/VLP-16.urdf.xacro"/>
+  <VLP-16 parent="base_link" name="velodyne" topic="/velodyne_points" hz="10" samples="440">
+    <origin xyz="0 0 ${chassis_height/2 + 0.075}" rpy="0 0 0" />
+  </VLP-16>
   <!-- Chassis -->
   <link name="chassis">
